File: Hardware/AK9750 Human Movement Sensor Breakout.sch (EAGLE design)
At the start: 25 parts, among them J2 SMD, J3 PTH, J4 SMD, U2 AK9750

Commit message: Changed sensor to AK9753
Parts:
- added JP10, JP9: FIDUCIALUFIDUCIAL, SparkFun:FIDUCIALUFIDUCIAL
- added LOGO3: REVISION, SparkFun-Aesthetics:REVISION
- J2, J4: value SMD -> Qwiic Right Angle; device SparkX:I2C_STANDARDJS-1MM -> SparkFun-Connectors:I2C_STANDARDQWIIC
- J3: device SparkX:I2C_STANDARD_NO_SILK -> SparkFun-Connectors:I2C_STANDARD_NO_SILK
- LOGO2: value SFE_LOGO_NAME_FLAME.1_INCH -> SFE_LOGO_NAME.1_INCH; device SparkFun-Aesthetics:SFE_LOGO_NAME_FLAME.1_INCH -> SparkFun-Aesthetics:SFE_LOGO_NAME.1_INCH
- U2: value AK9750 -> AK9753; device SparkX:AK9750 -> SparkFun-Sensors:AK9750"
Connections:
- net 3.3V: now also J2.2, J3.2, J4.2; no longer J2.VCC, J3.VCC, J4.VCC
- net GND: now also J2.1, J3.1, J4.1; no longer J2.GND, J3.GND, J4.GND
- net SCL: now also J2.4, J3.4, J4.4; no longer J2.SCL, J3.SCL, J4.SCL
- net SDA: now also J2.3, J3.3, J4.3; no longer J2.SDA, J3.SDA, J4.SDA
Other:
- note added: "A. England"
- note added: "ADR0"
- note added: "Interrupt Pullup"
- note added: "v01"
- note removed: "X11"
- moved on the sheet: C1
