File: Hardware/AK9753 Human Movement Sensor.brd (EAGLE design)
At the start: 25.4 x 25.4 mm, 30 parts, among them J2 Qwiic Right Angle, J3 PTH, J4 Qwiic Right Angle, U2 AK9753

Commit message: Fixed that route out
Routing:
- net 3.3V: track 76.6 -> 71.4 mm
- net !INT: track 22.8 -> 24.6 mm, vias 1 -> 3
Changed lines of the file:
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@@
 <setting verticaltext="up"/>
 </settings>
-<grid distance="0.05" unitdist="inch" unit="inch" style="lines" multiple="1" display="yes" altdistance="0.005" altunitdist="inch" altunit="inch"/>
+<grid distance="0.05" unitdist="inch" unit="inch" style="lines" multiple="1" display="yes" altdistance="0.0025" altunitdist="inch" altunit="inch"/>
 <layers>
 <layer number="1" name="Top" color="4" fill="1" visible="yes" active="yes"/>
@@
 <wire x1="6.088" y1="13.2" x2="6.096" y2="13.208" width="0.1778" layer="1"/>
 <contactref element="R6" pad="2"/>
-<wire x1="11.0744" y1="11.7856" x2="11.0744" y2="11.5824" width="0.1778" layer="1"/>
-<wire x1="11.0744" y1="11.5824" x2="11.557" y2="11.0998" width="0.1778" layer="1"/>
-<wire x1="11.557" y1="10.033" x2="11.557" y2="11.0998" width="0.1778" layer="1"/>
 <wire x1="20.32" y1="5.85" x2="19.423" y2="5.85" width="0.1778" layer="1"/>
 <wire x1="19.177" y1="6.096" x2="19.177" y2="8.89" width="0.1778" layer="1"/>
@@
 <wire x1="19.177" y1="8.89" x2="19.177" y2="9.525" width="0.1778" layer="1"/>
 <wire x1="17.78" y1="9.398" x2="17.78" y2="6.35" width="0.1778" layer="16"/>
-<wire x1="10.922" y1="11.938" x2="11.0744" y2="11.7856" width="0.1778" layer="1"/>
 <wire x1="7.62" y1="11.85" x2="6.311" y2="11.85" width="0.1778" layer="1"/>
 <wire x1="6.311" y1="11.85" x2="6.096" y2="12.065" width="0.1778" layer="1"/>
@@
 <wire x1="10.475" y1="11.938" x2="8.89" y2="11.938" width="0.1778" layer="1"/>
 <wire x1="8.89" y1="11.938" x2="8.802" y2="11.85" width="0.1778" layer="1"/>
-<wire x1="10.475" y1="11.938" x2="10.922" y2="11.938" width="0.1778" layer="1"/>
-<wire x1="16.002" y1="10.414" x2="18.288" y2="10.414" width="0.1778" layer="1"/>
-<wire x1="11.557" y1="10.033" x2="11.2014" y2="9.6774" width="0.1778" layer="1"/>
-<wire x1="11.2014" y1="9.6774" x2="10.0584" y2="9.6774" width="0.1778" layer="1"/>
-<wire x1="10.0584" y1="9.6774" x2="9.906" y2="9.525" width="0.1778" layer="1"/>
-<wire x1="9.906" y1="9.525" x2="9.906" y2="8.929" width="0.1778" layer="1"/>
-<wire x1="9.906" y1="8.929" x2="9.945" y2="8.89" width="0.1778" layer="1"/>
 <wire x1="20.32" y1="16.9164" x2="22.86" y2="16.9164" width="0.1778" layer="1"/>
 <wire x1="6.35" y1="8.89" x2="6.35" y2="7.112" width="0.1778" layer="1"/>
 <wire x1="5.08" y1="6.85" x2="6.088" y2="6.85" width="0.1778" layer="1"/>
 <wire x1="6.088" y1="6.85" x2="6.35" y2="7.112" width="0.1778" layer="1"/>
-<wire x1="14.925" y1="10.638" x2="15.778" y2="10.638" width="0.1778" layer="1"/>
-<wire x1="15.778" y1="10.638" x2="16.002" y2="10.414" width="0.1778" layer="1"/>
 <wire x1="9.652" y1="14.732" x2="10.16" y2="15.24" width="0.1778" layer="1"/>
 <wire x1="10.16" y1="15.24" x2="12.065" y2="15.24" width="0.1778" layer="1"/>
@@
 <wire x1="17.78" y1="6.35" x2="12.7" y2="6.35" width="0.1778" layer="16"/>
 <wire x1="12.7" y1="8.128" x2="12.7" y2="6.35" width="0.1778" layer="16"/>
+<wire x1="16.7005" y1="10.414" x2="18.288" y2="10.414" width="0.1778" layer="1"/>
+<wire x1="16.7005" y1="10.414" x2="16.4765" y2="10.638" width="0.1778" layer="1"/>
+<wire x1="16.4765" y1="10.638" x2="14.925" y2="10.638" width="0.1778" layer="1"/>
+<wire x1="10.16" y1="8.89" x2="9.945" y2="8.89" width="0" layer="19" extent="1-16"/>
 </signal>
 <signal name="GND">
@@
 <via x="8.89" y="13.97" extent="1-16" drill="0.381"/>
 <via x="19.685" y="10.668" extent="1-16" drill="0.381"/>
-<via x="16.4592" y="8.89" extent="1-16" drill="0.381"/>
+<via x="16.1417" y="9.906" extent="1-16" drill="0.381"/>
 <via x="22.1742" y="8.89" extent="1-16" drill="0.381"/>
 </signal>
@@
 <contactref element="U2" pad="4"/>
 <contactref element="R2" pad="2"/>
-<wire x1="14.5392" y1="11.288" x2="14.224" y2="10.9728" width="0.1778" layer="1"/>
-<wire x1="14.925" y1="11.288" x2="15.89" y2="11.288" width="0.1778" layer="1"/>
-<wire x1="15.89" y1="11.288" x2="16.256" y2="10.922" width="0.1778" layer="1"/>
-<wire x1="14.925" y1="11.288" x2="14.5392" y2="11.288" width="0.1778" layer="1"/>
+<wire x1="14.925" y1="11.288" x2="16.4615" y2="11.288" width="0.1778" layer="1"/>
 <wire x1="21.59" y1="11.85" x2="21.59" y2="10.287" width="0.1778" layer="1"/>
 <wire x1="21.59" y1="10.287" x2="21.336" y2="10.033" width="0.1778" layer="1"/>
 <wire x1="21.336" y1="10.033" x2="19.304" y2="10.033" width="0.1778" layer="1"/>
 <wire x1="19.304" y1="10.033" x2="18.415" y2="10.922" width="0.1778" layer="1"/>
-<wire x1="18.415" y1="10.922" x2="16.256" y2="10.922" width="0.1778" layer="1"/>
-<wire x1="14.224" y1="10.9728" x2="14.224" y2="10.033" width="0.1778" layer="1"/>
-<wire x1="14.224" y1="10.033" x2="14.478" y2="9.779" width="0.1778" layer="1"/>
-<wire x1="14.478" y1="9.779" x2="14.478" y2="8.128" width="0.1778" layer="1"/>
-<wire x1="14.478" y1="8.128" x2="13.97" y2="7.62" width="0.1778" layer="1"/>
-<wire x1="13.97" y1="7.62" x2="10.16" y2="7.62" width="0.1778" layer="1"/>
+<wire x1="16.1925" y1="7.62" x2="10.16" y2="7.62" width="0.1778" layer="1"/>
 <via x="10.16" y="7.62" extent="1-16" drill="0.381"/>
 <wire x1="10.16" y1="7.62" x2="8.89" y2="7.62" width="0.1778" layer="16"/>
 <wire x1="8.89" y1="7.62" x2="7.62" y2="6.35" width="0.1778" layer="16"/>
 <wire x1="7.62" y1="6.35" x2="7.62" y2="3.81" width="0.1778" layer="16"/>
+<via x="16.4615" y="11.288" extent="1-16" drill="0.381"/>
+<wire x1="16.4615" y1="11.288" x2="16.8275" y2="10.922" width="0.1778" layer="16"/>
+<wire x1="16.8275" y1="10.922" x2="16.8275" y2="8.255" width="0.1778" layer="16"/>
+<wire x1="16.8275" y1="8.255" x2="16.1925" y2="7.62" width="0.1778" layer="16"/>
+<via x="16.1925" y="7.62" extent="1-16" drill="0.381"/>
+<wire x1="18.415" y1="10.922" x2="16.8275" y2="10.922" width="0.1778" layer="1"/>
+<wire x1="16.8275" y1="10.922" x2="16.4615" y2="11.288" width="0.1778" layer="1"/>
 </signal>
 <signal name="N$1">
@@
 <contactref element="U2" pad="1"/>
 <wire x1="11.645" y1="8.89" x2="13.628" y2="8.89" width="0.1778" layer="1"/>
-<wire x1="14.925" y1="13.238" x2="14.3556" y2="13.238" width="0.1778" layer="1"/>
-<wire x1="13.843" y1="11.0998" x2="13.843" y2="10.287" width="0.1778" layer="1"/>
-<wire x1="14.3556" y1="13.238" x2="14.2494" y2="13.1318" width="0.1778" layer="1"/>
-<wire x1="14.2494" y1="13.1318" x2="14.2494" y2="11.5062" width="0.1778" layer="1"/>
-<wire x1="14.2494" y1="11.5062" x2="13.843" y2="11.0998" width="0.1778" layer="1"/>
 <wire x1="13.628" y1="8.89" x2="13.628" y2="10.072" width="0.1778" layer="1"/>
-<wire x1="13.628" y1="10.072" x2="13.843" y2="10.287" width="0.1778" layer="1"/>
+<wire x1="14.925" y1="13.238" x2="14.508" y2="13.238" width="0.1778" layer="1"/>
+<wire x1="14.508" y1="13.238" x2="14.2875" y2="13.0175" width="0.1778" layer="1"/>
+<wire x1="14.2875" y1="13.0175" x2="14.2875" y2="10.7315" width="0.1778" layer="1"/>
+<wire x1="14.2875" y1="10.7315" x2="13.628" y2="10.072" width="0.1778" layer="1"/>
 </signal>
 </signals>

Commit message: Pre Review commit
Parts:
- removed U$3: CWM 0.5 GI V1, openPIR-temp:LENS-CWM-0.5-GI-V1
- moved JP1 2.54 mm to (22.9, 16.5)
- moved JP5 2.54 mm to (20.3, 16.5)
- moved R1 1.90 mm to (17.8, 12.7)
- moved R3 1.90 mm to (19.7, 12.7)
Connections:
- net !INT: now also U2.7; no longer U2.4
- net 3.3V: now also U2.3, U2.6; no longer U2.5, U2.8
- net ADR0: now also U2.9; no longer U2.2
- net ADR1: now also U2.8; no longer U2.3
- net GND: now also U2.1, U2.2; no longer U2.10, U2.9
- net SCL: now also U2.4; no longer U2.7
- net SDA: now also U2.5; no longer U2.6
- net VDD: now also U2.10; no longer U2.1
Routing:
- net ADR0: track 7.82 -> 18.2 mm
- net SDA: track 37.2 -> 45.6 mm, vias 1 -> 3
- net SCL: track 50.5 -> 45.0 mm, vias 5 -> 6
- net ADR1: track 10.9 -> 16.2 mm
- net !INT: track 24.6 -> 27.6 mm
- net 3.3V: track 71.4 -> 69.6 mm
Other:
- board text removed: "Route"
- board text removed: "Route out"
- board text removed: "out"

Commit message: Post Design Review Changes
Parts:
- removed U$1: (no value), SparkFun-Aesthetics:ORDERING_INSTRUCTIONS
- moved J2 6.35 mm to (5.08, 12.7)
- moved J4 6.35 mm to (20.3, 12.7)
- moved R2 5.45 mm to (19.6, 7.62)
- moved R3 5.43 mm to (21.6, 7.62)
- moved J3 2.54 mm to (10.2, 1.27)
- moved J5 2.54 mm to (7.62, 1.27)
- moved JP5 2.01 mm to (18.4, 17.1)
- moved R4 1.91 mm to (15.9, 16.6)
- moved JP1 1.42 mm to (21.6, 17.1)
Routing:
- net ADR0: track 18.2 -> 28.5 mm, vias 0 -> 3
- net SDA: track 45.6 -> 53.1 mm
- net SCL: track 45.0 -> 38.0 mm
- net 3.3V: track 69.6 -> 64.7 mm
- net !INT: track 27.6 -> 24.8 mm, vias 3 -> 1
- net N$2: track 4.62 -> 2.74 mm
- net N$3: track 9.73 -> 11.5 mm
- net ADR1: track 16.2 -> 15.3 mm
Other:
- board text added: "v10"
- board text removed: "Rear mounted sensor requires 0.8mm thick PCB"
- board text removed: "v01"

Commit message: design review checklist
Parts:
- moved FRAME1 5.08 mm to (-15.2, -17.8)
- moved LOGO3 5.08 mm to (-3.81, -20.3)
Changed lines of the file:
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@@
 <layer number="27" name="tValues" color="7" fill="1" visible="no" active="yes"/>
 <layer number="28" name="bValues" color="7" fill="1" visible="no" active="yes"/>
-<layer number="29" name="tStop" color="7" fill="3" visible="no" active="yes"/>
+<layer number="29" name="tStop" color="7" fill="3" visible="yes" active="yes"/>
 <layer number="30" name="bStop" color="7" fill="6" visible="no" active="yes"/>
-<layer number="31" name="tCream" color="7" fill="4" visible="no" active="yes"/>
+<layer number="31" name="tCream" color="7" fill="4" visible="yes" active="yes"/>
 <layer number="32" name="bCream" color="7" fill="5" visible="no" active="yes"/>
 <layer number="33" name="tFinish" color="6" fill="3" visible="no" active="yes"/>
@@
 <layer number="45" name="Holes" color="7" fill="1" visible="no" active="yes"/>
 <layer number="46" name="Milling" color="3" fill="1" visible="no" active="yes"/>
-<layer number="47" name="Measures" color="7" fill="1" visible="no" active="yes"/>
+<layer number="47" name="Measures" color="7" fill="1" visible="yes" active="yes"/>
 <layer number="48" name="Document" color="7" fill="1" visible="no" active="yes"/>
 <layer number="49" name="Reference" color="7" fill="1" visible="no" active="yes"/>
 <layer number="50" name="dxf" color="7" fill="1" visible="no" active="yes"/>
-<layer number="51" name="tDocu" color="6" fill="1" visible="no" active="yes"/>
+<layer number="51" name="tDocu" color="6" fill="1" visible="yes" active="yes"/>
 <layer number="52" name="bDocu" color="7" fill="1" visible="no" active="yes"/>
 <layer number="53" name="tGND_GNDA" color="7" fill="9" visible="no" active="no"/>
@@
 <text x="18.4785" y="18.796" size="0.8128" layer="21" font="vector" ratio="15" align="center">0</text>
 <text x="21.6535" y="18.796" size="0.8128" layer="21" font="vector" ratio="15" align="center">1</text>
-<text x="10.16" y="-17.78" size="1.778" layer="51" font="vector">N. Seidle</text>
+<text x="15.24" y="-17.78" size="1.778" layer="51" font="vector">N. Seidle</text>
 <text x="12.7" y="23.495" size="1.016" layer="21" font="vector" ratio="15" rot="SR0" align="center">AK9753</text>
 <text x="12.573" y="22.098" size="1.016" layer="22" font="vector" ratio="15" rot="SMR0" align="center">Presence Sensor</text>
@@
 View
 </text>
-<text x="10.16" y="-20.32" size="1.778" layer="51" font="vector">A. England</text>
+<text x="15.24" y="-20.32" size="1.778" layer="51" font="vector">A. England</text>
 <text x="10.795" y="17.78" size="0.8128" layer="21" font="vector" ratio="15">I2C PU</text>
 <text x="19.812" y="10.033" size="0.8128" layer="22" font="vector" ratio="15" rot="MR270">JP8</text>
@@
 <attribute name="NAME" x="8.89" y="2.667" size="0.6096" layer="25" font="vector" ratio="20"/>
 </element>
-<element name="FRAME1" library="SparkFun-Aesthetics" package="CREATIVE_COMMONS" value="FRAME-LETTER" x="-20.32" y="-17.78"/>
+<element name="FRAME1" library="SparkFun-Aesthetics" package="CREATIVE_COMMONS" value="FRAME-LETTER" x="-15.24" y="-17.78"/>
 <element name="C4" library="SparkFun-Capacitors" package="0603" value="1.0uF" x="14.478" y="8.89" smashed="yes">
 <attribute name="PROD_ID" value="CAP-00868" x="14.478" y="8.89" size="1.778" layer="27" font="vector" ratio="15" display="off"/>
@@
 <element name="JP9" library="SparkFun" package="MICRO-FIDUCIAL" value="FIDUCIALUFIDUCIAL" x="0.762" y="24.638" rot="MR0"/>
 <element name="JP10" library="SparkFun" package="MICRO-FIDUCIAL" value="FIDUCIALUFIDUCIAL" x="24.511" y="0.889" rot="MR0"/>
-<element name="LOGO3" library="SparkFun-Aesthetics" package="REVISION" value="REVISION" x="-8.89" y="-20.32"/>
+<element name="LOGO3" library="SparkFun-Aesthetics" package="REVISION" value="REVISION" x="-3.81" y="-20.32"/>
 </elements>
 <signals>

Commit message: v10 fixes
Parts:
- J2, J4: value Qwiic Right Angle -> (none)
