File: Hardware/AK9753 Human Movement Sensor.sch (EAGLE design)
At the start: 28 parts, among them J2 Qwiic Right Angle, J3 PTH, J4 Qwiic Right Angle, U2 AK9753

Commit message: Pre Review commit
Parts:
- removed U$3: CWM 0.5 GI V1, openPIR-temp:PIR-LENSCWM-0.5-GI-V1
Changed lines of the file:
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@@
 <part name="R6" library="SparkFun-Resistors" deviceset="330OHM" device="-0603-1/10W-1%" value="330"/>
 <part name="SUPPLY10" library="SparkFun-PowerSymbols" deviceset="3.3V" device=""/>
-<part name="U$3" library="openPIR-temp" deviceset="PIR-LENS" device="CWM-0.5-GI-V1" value="CWM 0.5 GI V1"/>
 <part name="LOGO2" library="SparkFun-Aesthetics" deviceset="SFE_LOGO_NAME" device=".1_INCH"/>
 <part name="JP9" library="SparkFun" deviceset="FIDUCIAL" device="UFIDUCIAL"/>
@@
 <instance part="R6" gate="G$1" x="63.5" y="132.08" rot="R90"/>
 <instance part="SUPPLY10" gate="G$1" x="63.5" y="139.7"/>
-<instance part="U$3" gate="G$1" x="45.72" y="10.16"/>
 <instance part="LOGO2" gate="G$1" x="89.154" y="1.27"/>
 <instance part="JP9" gate="G$1" x="233.68" y="30.48"/>

Commit message: Post Design Review Changes
Other:
- note added: "v10"
- note removed: "v01"
Changed lines of the file:
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@@
 <plain>
 <text x="170.434" y="11.43" size="2.54" layer="94">N. Seidle</text>
-<text x="237.744" y="7.366" size="2.54" layer="94">v01</text>
+<text x="237.744" y="7.366" size="2.54" layer="94">v10</text>
 <text x="182.626" y="121.412" size="1.27" layer="97" align="center-left">Default 7-Bit Address: 0x64</text>
 <text x="185.928" y="117.856" size="1.27" layer="97" align="center-left">ADR0</text>

Commit message: v10 fixes
Parts:
- J2, J4: value Qwiic Right Angle -> (none); device SparkFun-Connectors:I2C_STANDARDQWIIC -> SparkFun-Connectors:QWIIC_CONNECTORJS-1MM
Changed lines of the file:
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@@
 <part name="SUPPLY4" library="SparkFun-PowerSymbols" deviceset="3.3V" device=""/>
 <part name="GND4" library="SparkFun" deviceset="GND" device=""/>
-<part name="J2" library="SparkFun-Connectors" deviceset="I2C_STANDARD" device="QWIIC" value="Qwiic Right Angle"/>
+<part name="J2" library="SparkFun-Connectors" deviceset="QWIIC_CONNECTOR" device="JS-1MM"/>
 <part name="GND6" library="SparkFun" deviceset="GND" device=""/>
 <part name="SUPPLY7" library="SparkFun-PowerSymbols" deviceset="3.3V" device=""/>
@@
 <part name="C4" library="SparkFun-Capacitors" deviceset="1.0UF" device="-0603-16V-10%" value="1.0uF"/>
 <part name="SUPPLY8" library="SparkFun-PowerSymbols" deviceset="3.3V" device=""/>
-<part name="J4" library="SparkFun-Connectors" deviceset="I2C_STANDARD" device="QWIIC" value="Qwiic Right Angle"/>
+<part name="J4" library="SparkFun-Connectors" deviceset="QWIIC_CONNECTOR" device="JS-1MM"/>
 <part name="GND8" library="SparkFun" deviceset="GND" device=""/>
 <part name="LOGO1" library="SparkFun-Aesthetics" deviceset="OSHW-LOGO" device="MINI"/>

Commit message: cleaned up repo, readme
Other:
- note added: "1 0 0x67"
- note removed: "1 0 0x66"
Changed lines of the file:
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@@
 <text x="196.85" y="117.856" size="1.27" layer="97" align="center-left">Address</text>
 <text x="187.96" y="113.284" size="1.27" layer="97" align="center-left">0   1    0x65</text>
-<text x="187.96" y="110.744" size="1.27" layer="97" align="center-left">1   0    0x66</text>
+<text x="187.96" y="110.744" size="1.27" layer="97" align="center-left">1   0    0x67</text>
 <text x="187.96" y="108.204" size="1.27" layer="97" align="center-left">1   1    Switch Mode</text>
 <text x="174.498" y="7.112" size="2.54" layer="94">A. England</text>
